File: _autosave-LightningReed.kicad_sch (KiCad schematic)
At the start: 14 parts, among them P1 Conn_WallPlug, Q1 Q_NMOS_GDS, U1 UCC28056

Commit message: File Sync
Parts:
- added R1: 10, symbol Device:R_Small
Connections:
- net at D3.2 (A), L4.1: now also Q1.2 (D)
- net at Q1.1 (G): now also R1.2
- net at U1.5 (DRV): now also R1.1
Other:
- moved on the sheet: Q1
Changed lines of the file:
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@@
   (junction (at 82.55 56.515) (diameter 0) (color 0 0 0 0)
   )
+  (junction (at 69.215 62.865) (diameter 0) (color 0 0 0 0)
+  )
   (wire (pts (xy 76.2 30.48) (xy 81.915 30.48))
     (stroke (width 0) (type default))
@@
     (stroke (width 0) (type default))
   )
+  (wire (pts (xy 69.215 62.865) (xy 71.12 62.865))
+    (stroke (width 0) (type default))
+  )
   (wire (pts (xy 27.305 56.515) (xy 31.115 56.515))
     (stroke (width 0) (type default))
@@
     (stroke (width 0) (type default))
   )
+  (wire (pts (xy 69.215 62.865) (xy 69.215 76.2))
+    (stroke (width 0) (type default))
+  )
+  (wire (pts (xy 36.195 81.28) (xy 36.195 97.79))
+    (stroke (width 0) (type default))
+  )
   (wire (pts (xy 49.53 34.29) (xy 49.53 33.02))
     (stroke (width 0) (type default))
@@
     (stroke (width 0) (type default))
   )
-  (wire (pts (xy 69.85 76.2) (xy 69.85 63.5))
-    (stroke (width 0) (type default))
-  )
-  (wire (pts (xy 67.31 62.865) (xy 71.12 62.865))
-    (stroke (width 0) (type default))
-  )
-  (wire (pts (xy 69.215 63.5) (xy 69.85 63.5))
+  (wire (pts (xy 55.245 81.28) (xy 36.195 81.28))
+    (stroke (width 0) (type default))
+  )
+  (wire (pts (xy 67.31 62.865) (xy 69.215 62.865))
     (stroke (width 0) (type default))
   )
@@
     (stroke (width 0) (type default))
   )
+  (wire (pts (xy 60.325 81.28) (xy 61.595 81.28))
+    (stroke (width 0) (type default))
+  )
   (wire (pts (xy 66.04 29.21) (xy 66.04 30.48))
     (stroke (width 0) (type default))
@@
   )
   (wire (pts (xy 42.545 56.515) (xy 45.085 56.515))
+    (stroke (width 0) (type default))
+  )
+  (wire (pts (xy 36.195 97.79) (xy 43.18 97.79))
     (stroke (width 0) (type default))
   )
@@
     )
   )
-  (symbol (lib_id "Device:Q_NMOS_GDS") (at 67.31 81.28 0) (unit 1)
-    (in_bom yes) (on_board yes) (dnp no) (fields_autoplaced)
-    (property "Reference" "Q1" (at 73.025 80.01 0)
-      (effects (font (size 1.27 1.27)) (justify left))
-    )
-    (property "Value" "Q_NMOS_GDS" (at 73.025 82.55 0)
-      (effects (font (size 1.27 1.27)) (justify left))
-    )
-    (property "Footprint" "" (at 72.39 78.74 0)
-      (effects (font (size 1.27 1.27)) hide)
-    )
-    (property "Datasheet" "~" (at 67.31 81.28 0)
-      (effects (font (size 1.27 1.27)) hide)
-    )
+  (symbol (lib_id "Device:R_Small") (at 57.785 81.28 90) (unit 1)
+    (in_bom yes) (on_board yes) (dnp no)
+    (property "Reference" "R1" (at 60.96 80.645 90)
+      (effects (font (size 0.8 0.8)))
+    )
+    (property "Value" "10" (at 57.785 81.28 90)
+      (effects (font (size 0.8 0.8)))
+    )
+    (property "Footprint" "" (at 57.785 81.28 0)
+      (effects (font (size 1.27 1.27)) hide)
+    )
+    (property "Datasheet" "~" (at 57.785 81.28 0)
+      (effects (font (size 1.27 1.27)) hide)
+    )
+    (pin "1")
+    (pin "2")
+    (instances
+      (project "LightningReed"
+        (path "/ed30a684-3009-4c45-ba04-268ec6465166"
+          (reference "R1") (unit 1)
+        )
+      )
+    )
+  )
+  (symbol (lib_id "Device:Q_NMOS_GDS") (at 66.675 81.28 0) (unit 1)
+    (in_bom yes) (on_board yes) (dnp no) (fields_autoplaced)
+    (property "Reference" "Q1" (at 72.39 80.01 0)
+      (effects (font (size 1.27 1.27)) (justify left))
+    )
+    (property "Value" "Q_NMOS_GDS" (at 72.39 82.55 0)
+      (effects (font (size 1.27 1.27)) (justify left))
+    )
+    (property "Footprint" "" (at 71.755 78.74 0)
+      (effects (font (size 1.27 1.27)) hide)
+    )
+    (property "Datasheet" "~" (at 66.675 81.28 0)
+      (effects (font (size 1.27 1.27)) hide)
+    )
