File: LightningReed.kicad_pcb (KiCad board)
At the start: 2 copper layers, 55 x 75 mm, 176 parts, among them P1 Conn_WallPlug, Q1 NCE65T180D, Q10 DMZ6005E, Q11 2N7002K, Q12 NCEP15T14D, Q13 BSS123, Q2 2N7002, Q3 1N60G, Q4 2N7002, Q5 2N7002K, Q6 2N7002K, Q7 CMSA65R280Q, Q8 CMSA65R280Q, Q9 NCE0102, T1 Transformer_2P_2S, U1 UCC28056, U2 78L05S, U3 LMC7111, U4 UCC28780, U5 UCC27712, U6 LM317LCPK, U7 FODM8801A, U8 TL431DBZ, U9 UCC24612-1DBV

Commit message: Finish
Parts:
- C28, C32, C33, C34, D11, D13, D14, Q10, R46, R48, R49, R50, R51, TH1: moved to B.Cu
- moved D11 62.1 mm to (117.1, 111.8)
- moved C28 58.9 mm to (113.8, 102.9), turned to 180 degrees
- moved TH1 46.2 mm to (125.0, 115.1)
- moved C33 45.0 mm to (124.7, 103.4), turned to 180 degrees
- moved R50 44.2 mm to (129.3, 109.0), turned to 90 degrees
- moved D13 41.9 mm to (140.2, 105.7)
- moved R51 40.2 mm to (130.8, 109.0), turned to 90 degrees
- moved C34 39.5 mm to (131.6, 105.9), turned to 180 degrees
- moved D14 39.4 mm to (143.0, 108.5), turned to 90 degrees
- moved R48 38.9 mm to (132.3, 109.0), turned to -90 degrees
- moved Q10 36.3 mm to (138.2, 124.5)
- moved Q11 32.7 mm to (146.8, 106.4)
- moved R46 31.0 mm to (133.3, 112.8), turned to -90 degrees
- moved R52 30.3 mm to (145.0, 103.9)
- moved C32 30.1 mm to (134.9, 112.8), turned to -90 degrees
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Routing:
- net GNDPWR: track 139.9 -> 207.4 mm, vias 48 -> 59
- net Net-(D14-K): track 0.00 -> 46.9 mm, vias 0 -> 2
- net Net-(D13-K): track 0.00 -> 38.3 mm, vias 0 -> 4
- net /VSV: track 2.29 -> 33.9 mm, vias 0 -> 3
- net /VDD3: track 35.2 -> 60.0 mm, vias 2 -> 4
- net /VSW: track 21.4 -> 45.9 mm, vias 0 -> 2
- net /RUN: track 0.00 -> 22.9 mm, vias 0 -> 1
- net /VREF: track 9.78 -> 18.4 mm, vias 0 -> 2
- net Net-(U4-NTC): track 0.00 -> 7.51 mm
- net VDD: track 25.8 -> 32.2 mm, vias 4 -> 5
- net /CTL: track 14.0 -> 19.0 mm, vias 1 -> 2
- net HT: track 88.7 -> 92.8 mm
- net Net-(Q11-D): track 0.00 -> 3.51 mm
- net /BUR: track 12.4 -> 15.8 mm
- net Net-(U4-VS): track 0.00 -> 3.26 mm
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- added copper zone on F.Cu, net VCOM
Other:
- board size 55 x 75 mm -> 55 x 76.5 mm
- board text added: "HIGH VOLTAGE WARNING DO NOT TOUCH WHILE WORKING"
