File: LightningReed.kicad_sch (KiCad schematic)
At the start: 163 parts, among them P1 Conn_WallPlug, Q1 NCE65T180D, Q10 DMZ6005E, Q11 2N7002K, Q12 NCEP15T14D, Q13 BSS123, Q2 2N7002, Q3 1N60G, Q4 2N7002, Q5 2N7002K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

Commit message: Finish
Connections:
- net VDD: now also C28.2, C29.2, D11.1 (K), U4.15 (VDD)
Changed lines of the file:
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@@
   (junction (at 220.345 95.25) (diameter 0) (color 0 0 0 0)
   )
+  (junction (at 199.39 98.425) (diameter 0) (color 0 0 0 0)
+  )
   (junction (at 71.12 34.29) (diameter 0) (color 0 0 0 0)
   )
@@
     (stroke (width 0) (type default))
   )
+  (wire (pts (xy 199.39 98.425) (xy 203.2 98.425))
+    (stroke (width 0) (type default))
+  )
   (wire (pts (xy 114.3 149.86) (xy 114.3 156.21))
     (stroke (width 0) (type default))
@@
     (stroke (width 0) (type default))
   )
+  (wire (pts (xy 197.485 98.425) (xy 199.39 98.425))
+    (stroke (width 0) (type default))
+  )
   (wire (pts (xy 53.34 165.1) (xy 53.34 148.59))
     (stroke (width 0) (type default))
@@
     (stroke (width 0) (type default))
   )
+  (wire (pts (xy 197.485 94.615) (xy 197.485 98.425))
+    (stroke (width 0) (type default))
+  )
   (wire (pts (xy 297.815 113.03) (xy 297.815 114.3))
     (stroke (width 0) (type default))
@@
     (stroke (width 0) (type default))
   )
-  (wire (pts (xy 199.39 98.425) (xy 203.2 98.425))
-    (stroke (width 0) (type default))
-  )
   (wire (pts (xy 81.915 98.425) (xy 76.835 98.425))
     (stroke (width 0) (type default))
@@
         )
       )
+    )
+  )
+  (symbol (lib_id "power:VDD") (at 197.485 94.615 0) (unit 1)
+    (in_bom yes) (on_board yes) (dnp no)
+    (property "Reference" "#PWR042" (at 197.485 98.425 0)
+      (effects (font (size 1.27 1.27)) hide)
+    )
+    (property "Value" "VDD" (at 196.215 97.79 90)
+      (effects (font (size 1.27 1.27)) (justify left))
+    )
+    (property "Footprint" "" (at 197.485 94.615 0)
+      (effects (font (size 1.27 1.27)) hide)
+    )
+    (property "Datasheet" "" (at 197.485 94.615 0)
+      (effects (font (size 1.27 1.27)) hide)
+    )
+    (pin "1")
+    (instances
+      (project "LightningReed"
+        (path "/ed30a684-3009-4c45-ba04-268ec6465166"
+          (reference "#PWR042") (unit 1)
+        )
+      )
